Commit message: Update mmo_700 URDFs and launch files

File: robots/mmo_700/urdf/mmo_700_body.urdf.xacro (robot description, xacro)
@@ -25,6 +25,6 @@
         <axis xyz="0 0 -1"/>
         <joint_properties damping="1" friction="1"/>
-        <parent link="base_footprint"/>
-        <child link="base_link"/>
+        <parent link="base_link"/>
+        <child link="base_footprint"/>
     </joint>
     <!-- Lidar Sensors -->

File: robots/mmo_700/urdf/mmo_700_gazebo.urdf.xacro (robot description, xacro)
@@ -15,5 +15,5 @@
         controller_update_rate="${controller_update_rate}"
         odom_frame="odom"
-        base_frame="base_footprint"
+        base_frame="base_link"
         covariance_yaw="0.0001"
     />
